Commit message: Set up initial positions. Still not segfaulting like it should

File: urdf/robot.urdf (robot description, URDF)
Before this commit: robot minimal_robot, 5 links, 4 joints
Joints:
- joint gripper_left_finger_joint: limit lower=0.0 upper=0.04 effort=50 velocity=0.5 -> lower=0.0 upper=0.05 effort=50 velocity=0.5
- joint gripper_right_finger_joint: axis 0 1 0 -> 0 -1 0; limit lower=-0.04 upper=0.0 effort=50 velocity=0.5 -> lower=0.0 upper=0.05 effort=50 velocity=0.5; mimic joint=gripper_left_finger_joint multiplier=-1 offset=0 -> joint=gripper_left_finger_joint multiplier=1 offset=0
- joint turntable_joint: limit lower=-3.14159 upper=3.14159 effort=100 velocity=1.0 -> lower=0.0 upper=6.2831853072 effort=100 velocity=1.0
